File: hardware/power_stage.kicad_sch (KiCad schematic)
At the start: 66 parts, among them J3 MOTOR, J9 BRAKE_RES, Q1 CSD19534Q5A, Q2 CSD19534Q5A, Q3 CSD19534Q5A, Q4 CSD19534Q5A, Q5 CSD19534Q5A, Q6 CSD19534Q5A, Q7 CSD19534Q5A, Q8 CSD19534Q5A, Q9 CSD19534Q5A, U3 DRV8300DPWR, U4 DRV8300DPWR, U5 INA240A2D, U6 INA240A2D

Commit message: Move HB3 to U3: U3 drives HB1-HB3, U4 drives HB4
BLDC (U/V/W = HB1-HB3) now runs on a single DRV8300; U4, Q7, Q8 and the
HB4 parts are marked with a Variant field for a DNP BLDC build. Optional
brake chopper moves to U4 channel B. DRV8300 symbol inputs reordered
(INL before INH) for clean GND ties. Handover K7/4.2, BOM and README updated.
Parts:
- C39, C41, C45, C53, C55, D8, D9, Q7, Q8, R35, R36, R39, R40, U4: Variant (none) -> STEP/DC only - DNP on single-driver BLDC build
Connections:
- net BRK_PWM: now also U4.5 (INLB); no longer U3.6 (INLC)
- net GH3: now also U3.13 (GHC); no longer U4.19 (GHA)
- net GH4: now also U4.19 (GHA); no longer U4.16 (GHB)
- net GL3: now also U3.9 (GLC); no longer U4.11 (GLA)
- net GL4: now also U4.11 (GLA); no longer U4.10 (GLB)
- net GL_BRK: now also U4.10 (GLB); no longer U3.9 (GLC)
- net GND: now also U4.2 (INHB); no longer U3.3 (INHC)
- net PH3: now also U3.12 (SHC); no longer U4.18 (SHA)
- net PH4: now also U4.18 (SHA); no longer U4.15 (SHB)
- net PWM_H3: now also U3.3 (INHC); no longer U4.1 (INHA)
- net PWM_H4: now also U4.1 (INHA); no longer U4.2 (INHB)
- net PWM_L3: now also U3.6 (INLC); no longer U4.4 (INLA)
- net PWM_L4: now also U4.4 (INLA); no longer U4.5 (INLB)
- net at C45.1: now also U4.20 (BSTA); no longer U4.17 (BSTB)
- net at C44.1: now also U3.14 (BSTC); no longer U4.20 (BSTA)
Other:
- note added: "U3 = HB1+HB2+HB3 (BLDC U/V/W on one driver). U4 = HB4 (+ optional brake chopper on ch. B). BLDC build: U4, Q7, Q8 + HB4 parts DNP. DRV8300D TSSOP: fixed 200 ns dead time + lockout."
- note removed: "DRV8300D TSSOP: fixed 200 ns dead time + cross-conduction lockout. MCU TIM1 DTG is a backup (50-100 ns). CBST <= 1 uF. U3 channel C: low side only -> optional brake chopper Q9 (DNP)."
- moved on the sheet: C44, C45
